File: BeagleBone-cape/pwr.kicad_sch (KiCad schematic)
At the start: 16 parts, among them IC1 A6983C50QTR

Commit message: Add i2c logic level translator
Parts:
- removed D3: D_Small, Diode_SMD:D_0603_1608Metric, symbol Device:D_Small
- added Q1: DMP3013SFV, Package_SON:Diodes_PowerDI3333-8, symbol Transistor_FET:DMP3013SFV
- added U6: LTC4412ES6, Package_TO_SOT_SMD:TSOT-23-6, symbol Power_Management:LTC4412xS6
Connections:
- net +5V: now also IC1.7 (VOUT/FB), Q1.1 (S), Q1.2 (S), Q1.3 (S), U6.6 (SENSE)
- net GND: now also U6.2 (GND), U6.3 (CTL)
- net BUCK_OUT: now reaches C14.2, C15.2, C16.2, L1.2, R18.2
- net BUCK_OUT: now also Q1.5 (D), U6.1 (VIN); no longer IC1.7 (VOUT/FB)
- new net: Q1.4 (G), U6.5 (GATE)
- no-connect marks 0 -> 1

Commit message: Cape: finish IMU/baro schematic, PCB sync and cleanup
Schematic:
- remove cape EEPROM U1, SW1, TP1 (#4)
- PGOOD to P8.12 via 10k pull-up R27 (#10)
- PWR_FLAGs on root, VBUS renamed SYS_5V, GPIO2/3 renamed UART_RX/TX (#6, #12, #33)
- VBIAS of A6983 to BUCK_OUT (#34)
- BMP390 symbol moved to Cape_lib, MPN fixed BMP388 -> BMP390 (#13)
- LSM6DSV16X/IIS2MDC: add C49 10 uF decoupling, fix C48 value/MPN (datasheet audit)

PCB:
- sync from schematic, place U9, U10, C44-C49, R27
- remove stray IMU-area +3V3/IMU_INT1 copper, old +3V3 In2 pour, dangling copper (#17, #18)
- design rules: outer track 0.10 mm, edge clearance 0.3 mm, zone clearance 0.2 mm (#37)

Routing is not done: 46 unconnected pads remain for manual routing.
DRC: 1 courtyard overlap (R27/R18), 7 pre-existing lib_footprint_mismatch warnings.
Connections:
- net BUCK_OUT: now also IC1.6 (VBIAS)
- net GND: no longer IC1.6 (VBIAS)
Other:
- company: (none) -> Skylark
- title: (none) -> Skylark BeagleBone Black cape - power
Changed lines of the file:
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@@
 	(generator_version "9.0")
 	(paper "A4")
+	(title_block
+		(title "Skylark BeagleBone Black cape - power")
+		(date "2026-10-18")
+		(rev "2 (draft)")
+		(company "Skylark")
+		(comment 1 "24 V input, A6983 5 V buck, LTC4412 ideal diode")
+	)
 	(junction
 		(at 127 96.52)
@@
 	(symbol
 		(lib_id "power:GND")
-		(at 166.37 86.36 90)
-		(unit 1)
-		(exclude_from_sim no)
-		(in_bom yes)
-		(on_board yes)
-		(dnp no)
-		(fields_autoplaced yes)
-		(property "Reference" "#PWR0301"
-			(at 166.37 92.71 0)
-			(effects
-				(font
-					(size 1.27 1.27)
-				)
-				(hide yes)
-			)
-		)
-		(property "Value" "GND"
-			(at 170.18 86.36 0)
-			(effects
-				(font
-					(size 1.27 1.27)
-				)
-				(hide yes)
-			)
-		)
-		(property "Footprint" ""
-			(at 166.37 86.36 0)
-			(effects
-				(font
-					(size 1.27 1.27)
-				)
-				(hide yes)
-			)
-		)
-		(property "Datasheet" ""
-			(at 166.37 86.36 0)
-			(effects
-				(font
-					(size 1.27 1.27)
-				)
-				(hide yes)
-			)
-		)
-		(property "Description" "Power symbol creates a global label with name \"GND\" , ground"
-			(at 166.37 86.36 0)
-			(effects
-				(font
-					(size 1.27 1.27)
-				)
-				(hide yes)
-			)
-		)
-		(pin "1"
-		)
-		(instances
-			(project "BeagleBone-cape"
-				(path "/e63e39d7-6ac0-4ffd-8aa3-1841a4541b55/bd0b971e-2693-4cc8-ae48-079dcad29646"
-					(reference "#PWR0301")
-					(unit 1)
-				)
-			)
-		)
-	)
-	(symbol
-		(lib_id "power:GND")
 		(at 195.58 105.41 0)
 		(unit 1)
@@
 		)
 	)
+	(label "BUCK_OUT"
+		(at 166.37 86.36 0)
+		(effects
+			(font
+				(size 1.27 1.27)
+			)
+			(justify left bottom)
+		)
+	)

Commit message: Cape: add baro and IMU/mag schematic sheets, sync root/PCB/project files
Changed lines of the file:
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@@
 	(wire
 		(pts
-			(xy 163.83 86.36) (xy 166.37 86.36)
+			(xy 163.83 86.36) (xy 176.53 86.36)
 		)
 		(stroke
@@
 		)
 	)
+	(label "BUCK_OUT"
+		(at 176.53 86.36 180)
+		(effects
+			(font
+				(size 1.27 1.27)
+			)
+			(justify right bottom)
+		)
+	)
 	(hierarchical_label "+5V"
 		(shape output)
@@
 		)
 	)
-	(label "BUCK_OUT"
-		(at 166.37 86.36 0)
-		(effects
-			(font
-				(size 1.27 1.27)
-			)
-			(justify left bottom)
-		)
-	)
