File: BeagleBone-cape/pwr.kicad_sch (KiCad schematic)
At the start: 17 parts, among them IC1 A6983C50QTR, Q1 DMP3013SFV, U6 LTC4412ES6

Commit message: Cape schematic: input protection, buzzer fix, CAN GND/jumper, LCSC field, lib refresh; ISSUES rewrite
Co-Authored-By: Claude Sonnet 5.5 <noreply@anthropic.com>
Parts:
- added C31: 100u 50V, Capacitor_SMD:CP_Elec_8x10, symbol Device:C_Polarized_Small
- added C33, C34: 22u 25V, Capacitor_SMD:C_1206_3216Metric_Pad1.33x1.80mm_HandSolder, symbol Device:C_Small
- added D7: SMBJ33CA, Diode_SMD:D_SMB, symbol Device:D_TVS_Small
- added D8: BZT52C12, Diode_SMD:D_SOD-123, symbol Device:D_Zener_Small
- added Q3: AOD4185L, Package_TO_SOT_SMD:TO-252-2, symbol Transistor_FET:Q_PMOS_GDS
- added R29: 100k, Resistor_SMD:R_0603_1608Metric_Pad0.98x0.95mm_HandSolder, symbol Device:R_Small
- C10, C11, C8, C9: LCSC (none) -> C15849; LSCS Part Number C15849 -> (none)
- C12: value 10u -> 10u 50V; footprint Capacitor_SMD:C_0603_1608Metric_Pad1.08x0.95mm_HandSolder -> Capacitor_SMD:C_1206_3216Metric_Pad1.33x1.80mm_HandSolder; LCSC (none) -> C13585; LSCS Part Number C194427 -> (none); Link https://www.lcsc.com/product-detail/C194427.html -> https://www.lcsc.com/product-detail/C13585.html; Manufacturer_Name (none) -> Samsung Electro-Mechanics; Manufacturer_Part_Number GRM188R6YA106MA73D -> CL31A106KBHNNNE
- C13: LCSC (none) -> C14663; LSCS Part Number C14663 -> (none)
- C14, C15, C16: LCSC (none) -> C48935064; LSCS Part Number C48935064 -> (none)
- F1: value Fuse -> 2A 63V; footprint Fuse:Fuse_1812_4532Metric_Pad1.30x3.40mm_HandSolder -> Fuse:Fuse_1206_3216Metric_Pad1.42x1.75mm_HandSolder; LCSC (none) -> C3105; Link (none) -> https://www.lcsc.com/product-detail/C3105.html; Manufacturer_Name (none) -> Littelfuse; Manufacturer_Part_Number (none) -> 0466002.NRHF
- L1: LCSC (none) -> C5123035; LSCS Part Number C5123035 -> (none)
- R12: LCSC (none) -> C22978; LSCS Part Number C22978 -> (none)
- R13: LCSC (none) -> C105588; LSCS Part Number C105588 -> (none)
- R18: LCSC (none) -> C105578; LSCS Part Number C105578 -> (none)
Connections:
- net +24V: now also C31.1, D8.1 (K), Q3.3 (S); no longer F1.2
- net BUCK_OUT: now also C33.1, C34.1
- net GND: now also C31.2, C33.2, C34.2, D7.1 (A1), R29.2
- new net: D8.2 (A), Q3.1 (G), R29.1
- new net VIN_F: D7.2 (A2), F1.2, Q3.2 (D)
Other:
- moved on the sheet: F1

Commit message: WIP: Q3 -> S-LP03N060TZHG (SOT-223), PCB synced with new schematic parts, not yet routed (DRC: shorts, 200 unconnected)
Co-Authored-By: Claude Sonnet 5.5 <noreply@anthropic.com>
Parts:
- removed C33, C34: 22u 25V, Capacitor_SMD:C_1206_3216Metric_Pad1.33x1.80mm_HandSolder, symbol Device:C_Small
- Q3: value AOD4185L -> S-LP03N060TZHG; footprint Package_TO_SOT_SMD:TO-252-2 -> Package_TO_SOT_SMD:SOT-223-3_TabPin2; LCSC C77993 -> C5200150; Link https://www.lcsc.com/product-detail/C77993.html -> https://www.lcsc.com/product-detail/C5200150.html; Manufacturer_Name Alpha & Omega Semiconductor -> LRC; Manufacturer_Part_Number AOD4185L -> S-LP03N060TZHG

Commit message: WIP: snap servo/LED/motor connectors to 4x2 grid, further PCB and pwr sheet edits
Co-Authored-By: Claude Sonnet 5.5 <noreply@anthropic.com>
Parts:
- removed C12: 10u 50V, Capacitor_SMD:C_1206_3216Metric_Pad1.33x1.80mm_HandSolder, symbol Device:C_Small
Changed lines of the file:
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@@
 	)
 	(junction
-		(at 90.17 76.2)
-		(diameter 0)
-		(color 0 0 0 0)
-	)
-	(junction
 		(at 35.56 76.2)
 		(diameter 0)
@@
 	(wire
 		(pts
-			(xy 90.17 76.2) (xy 90.17 88.9)
-		)
-		(stroke
-			(width 0)
-			(type solid)
-		)
-	)
-	(wire
-		(pts
 			(xy 127 93.98) (xy 127 96.52)
 		)
@@
 	(wire
 		(pts
-			(xy 90.17 76.2) (xy 97.79 76.2)
-		)
-		(stroke
-			(width 0)
-			(type solid)
-		)
-	)
-	(wire
-		(pts
-			(xy 76.2 76.2) (xy 90.17 76.2)
+			(xy 76.2 76.2) (xy 97.79 76.2)
 		)
 		(stroke
@@
 	(wire
 		(pts
-			(xy 90.17 93.98) (xy 90.17 105.41)
-		)
-		(stroke
-			(width 0)
-			(type solid)
-		)
-	)
-	(wire
-		(pts
 			(xy 214.63 104.14) (xy 212.09 104.14)
 		)
@@
 	)
 	(symbol
-		(lib_id "Device:C_Small")
-		(at 90.17 91.44 180)
-		(unit 1)
-		(exclude_from_sim no)
-		(in_bom yes)
-		(on_board yes)
-		(dnp no)
-		(property "Reference" "C12"
-			(at 91.694 90.1635 0)
-			(effects
-				(font
-					(size 1.27 1.27)
-				)
-				(justify right)
-			)
-		)
-		(property "Value" "10u 50V"
-			(at 91.694 92.7035 0)
-			(effects
-				(font
-					(size 1.27 1.27)
-				)
-				(justify right)
-			)
-		)
-		(property "Footprint" "Capacitor_SMD:C_1206_3216Metric_Pad1.33x1.80mm_HandSolder"
-			(at 90.17 91.44 0)
-			(effects
-				(font
-					(size 1.27 1.27)
-				)
-				(hide yes)
-			)
-		)
-		(property "Datasheet" "~"
-			(at 90.17 91.44 0)
-			(effects
-				(font
-					(size 1.27 1.27)
-				)
-				(hide yes)
-			)
-		)
-		(property "Description" "Unpolarized capacitor, small symbol"
-			(at 90.17 91.44 0)
-			(effects
-				(font
-					(size 1.27 1.27)
-				)
-				(hide yes)
-			)
-		)
-		(property "LCSC" "C13585"
-			(at 90.17 91.44 0)
-			(effects
-				(font
-					(size 1.27 1.27)
-				)
-				(hide yes)
-			)
-		)
-		(property "Link" "https://www.lcsc.com/product-detail/C13585.html"
-			(at 90.17 91.44 0)
-			(effects
-				(font
-					(size 1.27 1.27)
-				)
-				(hide yes)
-			)
-		)
-		(property "Manufacturer_Part_Number" "CL31A106KBHNNNE"
-			(at 90.17 91.44 0)
-			(effects
-				(font
-					(size 1.27 1.27)
-				)
-				(hide yes)
-			)
-		)
-		(property "Manufacturer_Name" "Samsung Electro-Mechanics"
-			(at 90.17 91.44 0)
-			(effects
-				(font
-					(size 1.27 1.27)
-				)
-				(hide yes)
-			)
-		)
-		(pin "1"
-		)
-		(pin "2"
-		)
-		(instances
-			(project "BeagleBone-cape"
-				(path "/e63e39d7-6ac0-4ffd-8aa3-1841a4541b55/bd0b971e-2693-4cc8-ae48-079dcad29646"
-					(reference "C12")
-					(unit 1)
-				)
-			)
-		)
-	)
-	(symbol
 		(lib_id "power:GND")
 		(at 111.76 105.41 0)
@@
 					(unit 1)
 				)
-			)
-		)
-	)
-	(symbol
-		(lib_id "power:GND")
-		(at 90.17 105.41 0)
-		(unit 1)
-		(exclude_from_sim no)
-		(in_bom yes)
-		(on_board yes)
-		(dnp no)
-		(fields_autoplaced yes)
-		(property "Reference" "#PWR049"
-			(at 90.17 111.76 0)
-			(effects
-				(font
-					(size 1.27 1.27)
-				)
-				(hide yes)
-			)
-		)
-		(property "Value" "GND"
-			(at 90.17 110.49 0)
-			(effects
-				(font
-					(size 1.27 1.27)
-				)
-			)
-		)
-		(property "Footprint" ""
-			(at 90.17 105.41 0)
-			(effects
-				(font
-					(size 1.27 1.27)
-				)
-				(hide yes)
-			)
-		)
-		(property "Datasheet" ""
-			(at 90.17 105.41 0)
-			(effects
-				(font
-					(size 1.27 1.27)
-				)
-				(hide yes)
-			)
-		)
-		(property "Description" "Power symbol creates a global label with name \"GND\" , ground"
-			(at 90.17 105.41 0)
-			(effects
-				(font
-					(size 1.27 1.27)
-				)
-				(hide yes)
-			)
-		)
-		(pin "1"
-		)
-		(instances
-			(project "BeagleBone-cape"
-				(path "/e63e39d7-6ac0-4ffd-8aa3-1841a4541b55/bd0b971e-2693-4cc8-ae48-079dcad29646"
-					(reference "#PWR049")
-					(unit 1)
-				)
