File: BeagleBone-cape/BeagleBone-cape.kicad_pcb (KiCad board)
At the start: 4 copper layers, 86.4 x 54.6 mm, 102 parts, among them IC1 A6983C50QTR, IC2 TCAN3413DDFR, IC3 BMP390, J1 Servo 0, J10 MotorR, J11 CAN, J12 24V, J13 MAVLink, J2 Servo 1, J3 Servo 2, J4 Servo 3, J5 LEDL, J6 LEDR, J8 Air Speed Sensor, J9 MotorL, P8 BeagleBone_Black_Header, P9 BeagleBone_Black_Header, Q1 DMP3013SFV, Q2 Q_NMOS_GSD, U1 IIS2MDC, U2 LSM6DSV16X, U3 DS1307ZN+, U4 LSM6DSV16X, U6 LTC4412ES6, Y1 32.768kHz

Commit message: PCB: remove dangling +24V vias and SPI1.SCLK stubs; ISSUES: DRC status update
Routing:
- net +24V: track 28.9 -> 28.8 mm, vias 14 -> 12
Changed lines of the file:
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@@
 	)
 	(segment
-		(start 153.45 87.5325)
-		(end 153.45 87.5725)
-		(width 0.15)
-		(layer "F.Cu")
-		(net 62)
-	)
-	(segment
 		(start 153.605431 87.871677)
 		(end 153.45 87.716246)
@@
 	)
 	(segment
-		(start 153.538162 87.696826)
-		(end 153.45 87.608664)
-		(width 0.15)
-		(layer "In2.Cu")
-		(net 62)
-	)
-	(segment
 		(start 153.01 81.66)
 		(end 153.01 81.3125)
@@
 	)
 	(segment
-		(start 122.52 87.16)
-		(end 122.4 87.16)
-		(width 0.2)
-		(layer "F.Cu")
-		(net 72)
-	)
-	(segment
 		(start 119.5875 80.395)
 		(end 120.4075 79.575)
@@
 		(net 72)
 	)
-	(via
-		(at 121.92 87.16)
-		(size 0.45)
-		(drill 0.25)
-		(layers "F.Cu" "B.Cu")
-		(free yes)
-		(net 72)
-	)
-	(via
-		(at 122.52 87.16)
-		(size 0.45)
-		(drill 0.25)
-		(layers "F.Cu" "B.Cu")
-		(free yes)
-		(net 72)
-	)
