File: BeagleBone-cape/BeagleBone-cape.kicad_sch (KiCad schematic)
At the start: 61 parts, among them IC2 TCAN3413DDFR, J1 Servo 0, J10 MotorR, J11 CAN, J12 24V, J13 MAVLink, J2 Servo 1, J3 Servo 2, J4 Servo 3, J5 LEDL, J6 LEDR, J8 Air Speed Sensor, J9 MotorL, P8 BeagleBone_Black_Header, P9 BeagleBone_Black_Header, Q2 Q_NMOS_GSD, U3 DS1307ZN+, Y1 32.768kHz

Commit message: Cape: unify CAN/FDCAN net names in schematic; ISSUES: ERC/DRC status update
Co-Authored-By: Claude Sonnet 5.5 <noreply@anthropic.com>
Connections:
- net CAN+ renamed CANH
- net CAN- renamed CANL
Changed lines of the file:
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@@
 		)
 	)
-	(label "GPIO15"
-		(at 299.72 180.34 180)
-		(effects
-			(font
-				(size 1.27 1.27)
-			)
-			(justify right bottom)
-		)
-	)
 	(label "SPI1.D0"
 		(at 248.92 187.96 0)
@@
 		)
 	)
-	(label "CAN-"
+	(label "CANL"
 		(at 551.18 74.93 180)
 		(effects
@@
 		)
 	)
-	(label "GPIO14"
-		(at 299.72 182.88 180)
-		(effects
-			(font
-				(size 1.27 1.27)
-			)
-			(justify right bottom)
-		)
-	)
 	(label "SERVO_2"
 		(at 513.08 232.41 180)
@@
 		)
 	)
-	(label "CAN+"
+	(label "CANH"
 		(at 551.18 91.44 180)
 		(effects
@@
 	)
 	(symbol
-		(lib_id "power:PWR_FLAG")
-		(at 340.36 388.62 0)
-		(unit 1)
-		(exclude_from_sim no)
-		(in_bom yes)
-		(on_board yes)
-		(dnp no)
-		(fields_autoplaced yes)
-		(property "Reference" "#FLG0106"
-			(at 340.36 386.715 0)
-			(effects
-				(font
-					(size 1.27 1.27)
-				)
-				(hide yes)
-			)
-		)
-		(property "Value" "PWR_FLAG"
-			(at 340.36 383.54 0)
-			(effects
-				(font
-					(size 1.27 1.27)
-				)
-			)
-		)
-		(property "Footprint" ""
-			(at 340.36 388.62 0)
-			(effects
-				(font
-					(size 1.27 1.27)
-				)
-				(hide yes)
-			)
-		)
-		(property "Datasheet" "~"
-			(at 340.36 388.62 0)
-			(effects
-				(font
-					(size 1.27 1.27)
-				)
-				(hide yes)
-			)
-		)
-		(property "Description" "Special symbol for telling ERC where power comes from"
-			(at 340.36 388.62 0)
-			(effects
-				(font
-					(size 1.27 1.27)
-				)
-				(hide yes)
-			)
-		)
-		(pin "1"
-		)
-		(instances
-			(project "BeagleBone-cape"
-				(path "/e63e39d7-6ac0-4ffd-8aa3-1841a4541b55"
-					(reference "#FLG0106")
-					(unit 1)
-				)
-			)
-		)
-	)
-	(symbol
 		(lib_name "+5V_2")
 		(lib_id "power:+5V")
@@
 				)
 			)
+		)
+	)
+	(symbol
+		(lib_id "power:PWR_FLAG")
+		(at 340.36 388.62 0)
+		(unit 1)
+		(exclude_from_sim no)
+		(in_bom yes)
+		(on_board yes)
+		(dnp no)
+		(fields_autoplaced yes)
+		(property "Reference" "#FLG0106"
+			(at 340.36 386.715 0)
+			(effects
+				(font
+					(size 1.27 1.27)
+				)
+				(hide yes)
+			)
+		)
+		(property "Value" "PWR_FLAG"
+			(at 340.36 383.54 0)
+			(effects
+				(font
+					(size 1.27 1.27)
+				)
+			)
+		)
+		(property "Footprint" ""
+			(at 340.36 388.62 0)
+			(effects
+				(font
+					(size 1.27 1.27)
+				)
+				(hide yes)
+			)
+		)
+		(property "Datasheet" "~"
+			(at 340.36 388.62 0)
+			(effects
+				(font
+					(size 1.27 1.27)
+				)
+				(hide yes)
+			)
+		)
+		(property "Description" "Special symbol for telling ERC where power comes from"
+			(at 340.36 388.62 0)
+			(effects
+				(font
+					(size 1.27 1.27)
+				)
+				(hide yes)
+			)
+		)
+		(pin "1"
+		)
+		(instances
+			(project "BeagleBone-cape"
+				(path "/e63e39d7-6ac0-4ffd-8aa3-1841a4541b55"
+					(reference "#FLG0106")
+					(unit 1)
+				)
+			)
