File: BeagleBone-cape/BeagleBone-cape.kicad_sch (KiCad schematic)
At the start: 61 parts, among them IC2 TCAN3413DDFR, J1 Servo 0, J10 MotorR, J11 CAN, J12 24V, J13 MAVLink, J2 Servo 1, J3 Servo 2, J4 Servo 3, J5 LEDL, J6 LEDR, J8 Air Speed Sensor, J9 MotorL, P8 BeagleBone_Black_Header, P9 BeagleBone_Black_Header, Q2 Q_NMOS_GSD, U3 DS1307ZN+, Y1 32.768kHz

Commit message: Cape schematic: input protection, buzzer fix, CAN GND/jumper, LCSC field, lib refresh; ISSUES rewrite
Co-Authored-By: Claude Sonnet 5.5 <noreply@anthropic.com>
Parts:
- added C32: 470u 16V, Capacitor_SMD:CP_Elec_8x10, symbol Device:C_Polarized_Small
- added JP1: CAN_TERM, Jumper:SolderJumper-2_P1.3mm_Bridged_RoundedPad1.0x1.5mm, symbol Jumper:SolderJumper_2_Bridged
- added R28: 1k, Resistor_SMD:R_0603_1608Metric_Pad0.98x0.95mm_HandSolder, symbol Device:R_Small
- BT1: LCSC (none) -> C2979167; LSCS Part Number C2979167 -> (none)
- BZ1: LCSC (none) -> C76871; LSCS Part Number C76871 -> (none)
- C17, C18, C29, C30: LCSC (none) -> C14663; LSCS Part Number C14663 -> (none)
- D6: LCSC (none) -> C233494; LSCS Part Number C233494 -> (none)
- IC2: LCSC (none) -> C30111221; LSCS Part Number C30111221 -> (none)
- J11: footprint TerminalBlock:TerminalBlock_Xinya_XY308-2.54-2P_1x02_P2.54mm_Horizontal -> TerminalBlock:TerminalBlock_Xinya_XY308-2.54-3P_1x03_P2.54mm_Horizontal; symbol Connector:Screw_Terminal_01x02 -> Connector:Screw_Terminal_01x03
- J2: value Servo 1 -> Servo 2
- J3: value Servo 2 -> Servo 1
- Q2: LCSC (none) -> C82045; LSCS Part Number C82045 -> (none)
- R10: value 420 -> 100; LCSC (none) -> C105588; Link (none) -> https://www.lcsc.com/product-detail/C105588.html; Manufacturer_Part_Number (none) -> RC0603FR-07100RL
- R11: value 420 -> 470; LCSC (none) -> C23179; Link (none) -> https://www.lcsc.com/product-detail/C23179.html; Manufacturer_Part_Number (none) -> 0603WAF4700T5E
- R19: LCSC (none) -> C14675; LSCS Part Number C14675 -> (none)
- R22, R23: LCSC (none) -> C99782; LSCS Part Number C99782 -> (none)
- R24, R27: LCSC (none) -> C98220; LSCS Part Number C98220 -> (none)
- R7: LCSC (none) -> C22787; LSCS Part Number C22787 -> (none)
- U3: LCSC (none) -> C26858; LSCS Part Number C26858 -> (none)
- Y1: LCSC (none) -> C32346; LSCS Part Number C32346 -> (none)
Connections:
- net +5V: now also C32.1, R28.1
- net CANH: now also JP1.1 (A); no longer R7.2
- net GND: now also J11.3 (Pin_3), C32.2
- net at BZ1.2 (-), Q2.3 (D): now also R28.2
- net FDCAN_RX renamed CAN_RX
- net FDCAN_TX renamed CAN_TX
- new net: JP1.2 (B), R7.2
Other:
- moved on the sheet: R7

Commit message: WIP: Q3 -> S-LP03N060TZHG (SOT-223), PCB synced with new schematic parts, not yet routed (DRC: shorts, 200 unconnected)
Co-Authored-By: Claude Sonnet 5.5 <noreply@anthropic.com>
Parts:
- removed C32: 470u 16V, Capacitor_SMD:CP_Elec_8x10, symbol Device:C_Polarized_Small
