File: BeagleBone-cape/imu_mag.kicad_sch (KiCad schematic)
At the start: 14 parts, among them U1 IIS2MDC, U2 LSM6DSV16X, U4 LSM6DSV16X

Commit message: Cape schematic: input protection, buzzer fix, CAN GND/jumper, LCSC field, lib refresh; ISSUES rewrite
Co-Authored-By: Claude Sonnet 5.5 <noreply@anthropic.com>
Parts:
- C19, C20, C21, C3, C5, C7: LCSC (none) -> C14663; LSCS Part Number C14663 -> (none)
- C4: LCSC (none) -> C6119835; LSCS Part Number C6119835 -> (none)
- C6: LCSC (none) -> C19702; LSCS Part Number C19702 -> (none)
Changed lines of the file:
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@@
 			)
 		)
-		(property "LSCS Part Number" "C14663"
+		(property "LCSC" "C14663"
 			(at 200.66 38.1 0)
 			(effects
@@
 			)
 		)
-		(property "LSCS Part Number" "C14663"
+		(property "LCSC" "C14663"
 			(at 72.39 43.18 0)
 			(effects
@@
 			)
 		)
-		(property "LSCS Part Number" "C14663"
+		(property "LCSC" "C14663"
 			(at 82.55 43.18 0)
 			(effects
@@
 			)
 		)
-		(property "LSCS Part Number" "C19702"
+		(property "LCSC" "C19702"
 			(at 105.41 43.18 0)
 			(effects
@@
 			)
 		)
-		(property "LSCS Part Number" "C6119835"
+		(property "LCSC" "C6119835"
 			(at 74.93 60.96 0)
 			(effects
@@
 			)
 		)
-		(property "LSCS Part Number" "C14663"
+		(property "LCSC" "C14663"
 			(at 190.5 38.1 0)
 			(effects
@@
 			)
 		)
-		(property "LSCS Part Number" "C14663"
+		(property "LCSC" "C14663"
 			(at 274.32 38.1 0)
 			(effects
@@
 			)
 		)
-		(property "LSCS Part Number" "C14663"
+		(property "LCSC" "C14663"
 			(at 261.62 38.1 0)
 			(effects
